Commit message: URDF File with Inertia

File: description/robot_core.xacro (robot description, xacro)
@@ -1,4 +1,5 @@
 <?xml version="1.0"?>
 <robot xmlns:xacro="http://www.ros.org/wiki/xacro"  name="robot">
+    <!--FILES -->
     <xacro:include filename="inertial_macros.xacro"/>
     <!--COLORS -->
@@ -26,5 +27,4 @@
     <link name="chassis">
         <visual>
-            <origin xyz="0 0 0"/>
             <geometry>
                 <box size="0.3048 0.381 0.12065"/>
@@ -37,5 +37,7 @@
             </geometry>
         </collision>
-        <xacro:inertial_box mass="0.5"/>
+        <xacro:inertial_box mass="1.3040781" x="0.3048" y="0.381" z="0.12065">
+            <origin xyz="0 0 0" rpy="0 0 0"/>
+        </xacro:inertial_box>
     </link>
     <joint name="left_front_chassis_joint" type="fixed">
@@ -58,4 +60,7 @@
             </geometry>
         </collision>
+        <xacro:inertial_box mass="0.2857632" x="0.3048" y="0.0381" z="0.0381">
+            <origin xyz="-0.13335 0 0" rpy="0 0 0"/>
+        </xacro:inertial_box>
     </link>
     <joint name="right_front_chassis_joint" type="fixed">
@@ -78,4 +83,7 @@
             </geometry>
         </collision>
+        <xacro:inertial_box mass="0.2857632" x="0.3048" y="0.0381" z="0.0381">
+            <origin xyz="-0.13335 0 0" rpy="0 0 0"/>
+        </xacro:inertial_box>
     </link>
     <!--BACK WHEELS -->
@@ -100,4 +108,7 @@
             </geometry>
         </collision>
+        <xacro:inertial_box mass="0.816239471" x="0.0381" y="0.1905" z="0.0381">
+            <origin xyz="0 0.05715 0" rpy="0 0 0"/>
+        </xacro:inertial_box>
     </link>
     <joint name="right_back_corner_motor_joint" type="continuous">
@@ -121,4 +132,7 @@
             </geometry>
         </collision>
+        <xacro:inertial_box mass="0.816239471" x="0.0381" y="0.1905" z="0.0381">
+            <origin xyz="0 0.05715 0" rpy="0 0 0"/>
+        </xacro:inertial_box>
     </link>
     <joint name="left_back_wheel_joint" type= "continuous">
@@ -140,4 +154,7 @@
             </geometry>
         </collision>
+        <xacro:inertial_cylinder mass="0.272155" length="0.0889" radius="0.0762">
+            <origin xyz="0 0 0" rpy = "0 0 0"/>
+        </xacro:inertial_cylinder>
     </link>
     <joint name="right_back_wheel_joint" type= "continuous">
@@ -159,4 +176,7 @@
             </geometry>
         </collision>
+        <xacro:inertial_cylinder mass="0.272155" length="0.0889" radius="0.0762">
+            <origin xyz="0 0 0" rpy = "0 0 0"/>
+        </xacro:inertial_cylinder>
     </link>
     <!--MIDDLE WHEELS -->
@@ -180,4 +200,7 @@
             </geometry>
         </collision>
+        <xacro:inertial_box mass="0.10296547" x="0.0381" y="0.0381" z="0.1651">
+            <origin xyz="0 0 0.08255" rpy="0 0 0"/>
+        </xacro:inertial_box>
     </link>
     <joint name="right_middle_diagonal_joint" type="fixed">
@@ -200,4 +223,7 @@
             </geometry>
         </collision>
+        <xacro:inertial_box mass="0.10296547" x="0.0381" y="0.0381" z="0.1651">
+            <origin xyz="0 0 0.08255" rpy="0 0 0"/>
+        </xacro:inertial_box>
     </link>
     <joint name="left_middle_balancer_joint" type="continuous">
@@ -221,4 +247,7 @@
             </geometry>
         </collision>
+        <xacro:inertial_box mass="0.469818593774" x="0.27305" y="0.0381" z="0.0381">
+            <origin xyz="-0.00635 0 0" rpy="0 0 0"/>
+        </xacro:inertial_box>
     </link>
     <joint name="right_middle_balancer_joint" type="continuous">
@@ -242,4 +271,7 @@
             </geometry>
         </collision>
+        <xacro:inertial_box mass="0.469818593774" x="0.27305" y="0.0381" z="0.0381">
+            <origin xyz="-0.00635 0 0" rpy="0 0 0"/>
+        </xacro:inertial_box>
     </link>
     <joint name="left_middle_wheel_joint" type= "continuous">
@@ -263,4 +295,7 @@
             </geometry>
         </collision>
+        <xacro:inertial_cylinder mass="0.272155" length="0.0889" radius="0.0762">
+            <origin xyz="0 0 0.0445" rpy = "0 0 0"/>
+        </xacro:inertial_cylinder>
     </link>
     <joint name="right_middle_wheel_joint" type= "continuous">
@@ -284,4 +319,7 @@
             </geometry>
         </collision>
+        <xacro:inertial_cylinder mass="0.272155" length="0.0889" radius="0.0762">
+            <origin xyz="0 0 0.0445" rpy = "0 0 0"/>
+        </xacro:inertial_cylinder>
     </link>
     <!--FRONT WHEELS -->
@@ -305,4 +343,7 @@
             </geometry>
         </collision>
+        <xacro:inertial_box mass="0.14424237" x="0.17145" y="0.0381" z="0.0381">
+            <origin xyz="0.066675 0 0" rpy="0 0 0"/>
+        </xacro:inertial_box>
     </link>
     <joint name="right_front_bar_joint" type= "fixed">
@@ -325,4 +366,7 @@
             </geometry>
         </collision>
+        <xacro:inertial_box mass="0.14424237" x="0.17145" y="0.0381" z="0.0381">
+            <origin xyz="0.066675 0 0" rpy="0 0 0"/>
+        </xacro:inertial_box>
     </link>
     <joint name="left_front_corner_motor_joint" type="continuous">
@@ -346,4 +390,7 @@
             </geometry>
         </collision>
+        <xacro:inertial_box mass="0.816239471" x="0.0381" y="0.1905" z="0.0381">
+            <origin xyz="0 0.05715 0" rpy="0 0 0"/>
+        </xacro:inertial_box>
     </link>
     <joint name="right_front_corner_motor_joint" type="continuous">
@@ -367,4 +414,7 @@
             </geometry>
         </collision>
+        <xacro:inertial_box mass="0.816239471" x="0.0381" y="0.1905" z="0.0381">
+            <origin xyz="0 0.05715 0" rpy="0 0 0"/>
+        </xacro:inertial_box>
     </link>
     <joint name="left_front_wheel_joint" type= "continuous">
@@ -386,4 +436,7 @@
             </geometry>
         </collision>
+        <xacro:inertial_cylinder mass="0.272155" length="0.0889" radius="0.0762">
+            <origin xyz="0 0 0" rpy = "0 0 0"/>
+        </xacro:inertial_cylinder>
     </link>
     <joint name="right_front_wheel_joint" type= "continuous">
@@ -405,4 +458,7 @@
             </geometry>
         </collision>
+        <xacro:inertial_cylinder mass="0.272155" length="0.0889" radius="0.0762">
+            <origin xyz="0 0 0" rpy = "0 0 0"/>
+        </xacro:inertial_cylinder>
     </link>
 </robot>
